Commit message: config_updates

File: localization/SLAM/LIO-SAM/config/robot.urdf.xacro (robot description, xacro)
@@ -2,5 +2,5 @@
 <robot name="lio" xmlns:xacro="http://tixiaoshan.github.io/">
   <xacro:property name="PI" value="3.1415926535897931" />
-  <link name="chassis_link"></link>
+  <!-- <link name="chassis_link"></link> -->
   <link name="base_link"></link>
   <joint name="base_link_joint" type="fixed">
@@ -9,27 +9,27 @@
     <origin xyz="0 0 0" rpy="0 0 0" />
   </joint>
-  <link name="lidar_link"> </link>
+  <link name="os_sensor"> </link>
   <joint name="lidar_joint" type="fixed">
+    <parent link="chassis_link" />
+    <child link="os_sensor" />
+    <origin xyz="0 0 2.5" rpy="0 0 0" />
+  </joint>
+  <link name="chassis_link"> </link>
+  <joint name="chassis_joint" type="fixed">
     <parent link="base_link" />
-    <child link="lidar_link" />
+    <child link="chassis_link" />
     <origin xyz="0 0 0" rpy="0 0 0" />
   </joint>
-  <link name="imu_link"> </link>
+  <link name="imu"> </link>
   <joint name="imu_joint" type="fixed">
     <parent link="chassis_link" />
-    <child link="imu_link" />
+    <child link="imu" />
     <origin xyz="0 0 0" rpy="0 0 0" />
   </joint>
-  <link name="laser_sensor_frame"> </link>
-  <joint name="laser_joint" type="fixed">
-    <parent link="imu_link" />
-    <child link="laser_sensor_frame" />
-    <origin xyz="0 0 0" rpy="0 0 0" />
-  </joint>
-  <link name="navsat_link"> </link>
+  <!-- <link name="navsat_link"> </link>
   <joint name="navsat_joint" type="fixed">
     <parent link="chassis_link" />
     <child link="navsat_link" />
     <origin xyz="0 0 0" rpy="0 0 0" />
-  </joint>
+  </joint> -->
 </robot>
